Commit message: Moved the front kinect

File: simulation_2017/urdf/cr17.xacro (robot description, xacro)
@@ -49,4 +49,8 @@
   <xacro:property name="scoopactmountback" value="0.03" /> <!-- get actual value -->
   <xacro:property name="scoopactmountin" value="${oneinch*8}" /> <!--based on the drawing having the center line of the actuator and inch past the offset, doublecheck-->
+  <xacro:property name="fronthorizontalsupportcontrolsboxoffset" value="${oneinch*8.5}" />
+  <xacro:property name="fronthorizontalsupportlength" value="${oneinch*18}" />
+  <xacro:property name="fronthorizontalsupportwidth" value="${oneinch}" />
+  <xacro:property name="fronthorizontalsupportheight" value="${oneinch*2}" />
   <xacro:property name="lidarmountheight" value="0.1" /> <!--get an actual value-->
   <xacro:property name="hokuyolength" value="0.04" /><!--get an actual value-->
@@ -573,4 +577,18 @@
   </joint>
   <xacro:kinect prefix="rear" parentlink="rear_kinect_mount"/>
+    <xacro:property name="fronthorizontalsupportcontrolsboxoffset" value="${oneinch*8.5}" />
+  <link name="front_horizontal_support">
+    <visual>
+      <geometry>
+        <box size="${fronthorizontalsupportwidth} ${fronthorizontalsupportlength} ${fronthorizontalsupportheight}" />
+      </geometry>
+      <material name="green"/>
+    </visual>
+  </link>
+  <joint name="to_front_horizontal_support" type="fixed">
+    <parent link="base_link"/>
+    <child link="front_horizontal_support"/>
+    <origin xyz="${fronthorizontalsupportcontrolsboxoffset+controlsboxlength/2} 0 -${controlsboxheight/2+fronthorizontalsupportheight/2}" />
+  </joint>
   <link name="front_kinect_mount">
     <visual>
@@ -582,7 +600,10 @@
   </link>
   <joint name="to_front_kinect_mount" type="fixed">
-    <parent link="base_link" />
+    <!-- We need to move the front kinect, this is so we can switch between the original position and the proposed new location for tests-->
+    <!--<parent link="base_link" />
+    <origin xyz="${controlsboxlength/2} 0 ${controlsboxheight/2+oneinch/2}" rpy="0 0 0"/>-->
+    <parent link="front_horizontal_support" />
+    <origin xyz="0 0 ${fronthorizontalsupportheight/2+oneinch/2}" rpy="0 0 0"/>
     <child link="front_kinect_mount"/>
-    <origin xyz="${controlsboxlength/2} 0 ${controlsboxheight/2+oneinch/2}" rpy="0 0 0"/>
   </joint>
   <xacro:kinect prefix="front" parentlink="front_kinect_mount"/>

Commit message: initial setup of nav stack, only test was that the launch file didn't crash and showed the map correctly in rviz

File: simulation_2017/urdf/cr17.xacro (robot description, xacro)
@@ -15,8 +15,8 @@
   <xacro:property name="armbaselength" value="${oneinch*2}" />
   <xacro:property name="armbasewidth" value="${oneinch}" />
-  <xacro:property name="armbaseheight" value="${oneinch*19}" />
+  <xacro:property name="armbaseheight" value="${oneinch*7}" />
   <xacro:property name="controlsboxlength" value="${oneinch*14.25}" />
   <xacro:property name="controlsboxwidth" value="${oneinch*18}" />
-  <xacro:property name="controlsboxheight" value="${oneinch*14}" />
+  <xacro:property name="controlsboxheight" value="${oneinch*7}" />
   <xacro:property name="wheeldiam" value="${oneinch*12}" />
   <xacro:property name="wheelwidth" value="${oneinch*3}" />
@@ -577,5 +577,4 @@
   </joint>
   <xacro:kinect prefix="rear" parentlink="rear_kinect_mount"/>
-    <xacro:property name="fronthorizontalsupportcontrolsboxoffset" value="${oneinch*8.5}" />
   <link name="front_horizontal_support">
     <visual>

Commit message: I think the transforms now work

File: simulation_2017/urdf/cr17.xacro (robot description, xacro)
@@ -15,8 +15,8 @@
   <xacro:property name="armbaselength" value="${oneinch*2}" />
   <xacro:property name="armbasewidth" value="${oneinch}" />
-  <xacro:property name="armbaseheight" value="${oneinch*7}" />
+  <xacro:property name="armbaseheight" value="${oneinch*19}" />
   <xacro:property name="controlsboxlength" value="${oneinch*14.25}" />
   <xacro:property name="controlsboxwidth" value="${oneinch*18}" />
-  <xacro:property name="controlsboxheight" value="${oneinch*7}" />
+  <xacro:property name="controlsboxheight" value="${oneinch*14}" />
   <xacro:property name="wheeldiam" value="${oneinch*12}" />
   <xacro:property name="wheelwidth" value="${oneinch*3}" />

Commit message: Updated the scoop size
Since we have the scoop, the actual size has been put in

File: simulation_2017/urdf/cr17.xacro (robot description, xacro)
@@ -38,6 +38,6 @@
   <xacro:property name="scooplinactmountbarlength" value="${oneinch*3}" />
   <xacro:property name="scooplinactmountbaroffset" value="${oneinch*7}" />
-  <xacro:property name="scooplength" value="0.2" /> <!--get actual value -->
-  <xacro:property name="scoopheight" value="0.3" /> <!--get actual value -->
+  <xacro:property name="scooplength" value="${oneinch*8.6875}" />
+  <xacro:property name="scoopheight" value="${oneinch*9.6875}" />
   <xacro:property name="scoopwidth" value="${oneinch*18}" />
   <xacro:property name="scoopdistancefromaxis" value="0.03" /> <!--get actual value -->
